File: PCB design/_autosave-Home.kicad_sch (KiCad schematic)
At the start: 22 parts, among them J1 Fan, J2 LCD, J3 EM lock, J4 ACS712 Signal, J5 Power In, J6 LCD, J7 RFID, J8 RFID, K1 SANYOU_SRD_Form_C, SW1 SW_SPST, U1 ACS712, U3 DHT11, U5 PIR, U6 MQ2

Commit message: final edits
Connections:
- net +3.3V: now also C1.1
- net 3V3: no longer C1.1
Changed lines of the file:
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@@
-    (stroke (width 0) (type default))
-  )
-  (wire (pts (xy 62.23 35.56) (xy 64.77 35.56))
     (stroke (width 0) (type default))
   )
@@
     (stroke (width 0) (type default))
   )
+  (wire (pts (xy 64.77 24.13) (xy 64.77 48.26))
+    (stroke (width 0) (type default))
+  )
   (wire (pts (xy 229.87 140.97) (xy 219.71 140.97))
     (stroke (width 0) (type default))
@@
   )
   (wire (pts (xy 115.57 97.79) (xy 106.68 97.79))
-    (stroke (width 0) (type default))
-  )
-  (wire (pts (xy 64.77 48.26) (xy 64.77 35.56))
     (stroke (width 0) (type default))
   )
@@
   )
   (wire (pts (xy 236.22 133.35) (xy 236.22 130.81))
+    (stroke (width 0) (type default))
+  )
+  (wire (pts (xy 43.18 24.13) (xy 64.77 24.13))
     (stroke (width 0) (type default))
   )
@@
     )
   )
-  (global_label "3V3" (shape output) (at 64.77 35.56 0) (fields_autoplaced)
+  (global_label "3V3" (shape output) (at 62.23 35.56 0) (fields_autoplaced)
     (effects (font (size 1.27 1.27)) (justify left))
-    (property "Intersheetrefs" "${INTERSHEET_REFS}" (at 71.1834 35.56 0)
+    (property "Intersheetrefs" "${INTERSHEET_REFS}" (at 68.6434 35.56 0)
       (effects (font (size 1.27 1.27)) (justify left) hide)
     )
